File: KeyboardPCB.kicad_pcb (KiCad board)
At the start: 2 copper layers, 399 x 117.7 mm, 236 parts

Commit message: routed switches
Parts:
- moved R_RESET1 2.59 mm to (127.4, 79.5), turned to 270 degrees
- moved D0:5 1.93 mm to (70.4, -5.08)
- moved C_UCAP1 0.63 mm to (132.3, 82.5), turned to 270 degrees
- moved Y_CLOCK1 0.33 mm to (142.1, 72.8), turned to 270 degrees
- turned C:1_CLOCK2 to 90 degrees
Routing:
- net COL2: track 0.00 -> 676.0 mm, vias 0 -> 56
- net COL0: track 0.00 -> 604.0 mm, vias 0 -> 12
- net COL1: track 0.00 -> 597.9 mm, vias 0 -> 60
- net COL3: track 0.00 -> 522.8 mm, vias 0 -> 46
- net COL5: track 0.00 -> 488.4 mm, vias 0 -> 38
- net COL4: track 0.00 -> 484.8 mm, vias 0 -> 40
- net COL6: track 0.00 -> 428.9 mm, vias 0 -> 26
- net COL7: track 0.00 -> 346.0 mm, vias 0 -> 22
- net COL8: track 0.00 -> 297.8 mm, vias 0 -> 18
- net COL9: track 0.00 -> 265.0 mm, vias 0 -> 10
- net ROW4: track 0.00 -> 232.6 mm, vias 0 -> 2
- net ROW7: track 0.00 -> 211.1 mm
- net ROW3: track 0.00 -> 201.1 mm, vias 0 -> 2
- net ROW9: track 0.00 -> 193.1 mm
- net ROW5: track 0.00 -> 190.9 mm, vias 0 -> 2
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Other:
- net class Default: trace_width 0.25 -> 0.254
- net class Power added: clearance 0.2, trace_width 0.381, via_dia 0.8, via_drill 0.4

Commit message: Routing
Parts:
- moved SW_RESET1 56.0 mm to (184.4, 81.8)
- moved R_RESET1 52.0 mm to (179.3, 77.2)
- moved C_UCAP1 0.68 mm to (132.6, 81.9)
- moved Y_CLOCK1 0.40 mm to (142.5, 72.9), turned to 180 degrees
- moved C:1_CLOCK2 0.38 mm to (138.3, 72.9), turned to 270 degrees
Routing:
- net GND: track 48.4 -> 260.0 mm, vias 0 -> 6
- net +5V: track 157.3 -> 328.5 mm, vias 2 -> 8
- net Net-(CONT1-Pad13): track 21.5 -> 85.6 mm, vias 0 -> 10
- net COL4: track 484.8 -> 523.2 mm, vias 40 -> 42
- net Net-(D9:0-Pad2): track 0.00 -> 10.9 mm
- net Net-(D3:6-Pad2): track 0.00 -> 10.9 mm
- net Net-(D8:4-Pad2): track 0.00 -> 10.8 mm
- net Net-(D8:5-Pad2): track 0.00 -> 10.8 mm
- net Net-(D3:4-Pad2): track 0.00 -> 10.8 mm
- net Net-(D9:1-Pad2): track 0.00 -> 10.8 mm
- net Net-(D8:1-Pad2): track 0.00 -> 10.8 mm
- net Net-(D3:5-Pad2): track 0.00 -> 10.7 mm
- net Net-(D8:7-Pad2): track 0.00 -> 10.7 mm
- net Net-(D3:7-Pad2): track 0.00 -> 10.7 mm
- net Net-(D9:8-Pad2): track 0.00 -> 10.6 mm
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
Commit message: Corrected pads, rerouting start
Parts:
- MX10:4_RSH1: footprint MX_Alps_Hybrid:MX-1U-NoLED -> MX_Alps_Hybrid:MX-2.75U-NoLED
- MX2:3_NU+1, MX4:3_NEN1, MX5:0_NU0, MX7:2_BSP1: footprint MX_Alps_Hybrid:MX-1U-NoLED -> MX_Alps_Hybrid:MX-2U-NoLED
- MX2:4_TAB1, MX8:2_\1: footprint MX_Alps_Hybrid:MX-1U-NoLED -> MX_Alps_Hybrid:MX-1.5U-NoLED
- MX3:4_CAP1: footprint MX_Alps_Hybrid:MX-1U-NoLED -> MX_Alps_Hybrid:MX-1.75U-NoLED
- MX4:4_LSH1, MX9:3_ENT1: footprint MX_Alps_Hybrid:MX-1U-NoLED -> MX_Alps_Hybrid:MX-2.25U-NoLED
- MX5:3_LCT1, MX5:4_OS1, MX5:5_LAL1: footprint MX_Alps_Hybrid:MX-1U-NoLED -> MX_Alps_Hybrid:MX-1.25U-NoLED
- MX5:9_SPC1: footprint MX_Alps_Hybrid:MX-1U-NoLED -> MX_Alps_Hybrid:MX-6.25U-NoLED
- moved R:HWB1 35.0 mm to (153.4, 122.6)
- moved C:DCP1 35.0 mm to (135.5, 112.1)
- moved C:DCP0 35.0 mm to (153.6, 113.9)
- moved C:DCP2 35.0 mm to (147.8, 126.7)
- moved C:DCP3 35.0 mm to (140.8, 126.7)
- moved CONT1 35.0 mm to (144.4, 117.7)
- moved C_UCAP1 35.0 mm to (135.0, 116.8)
- moved R_RESET1 31.1 mm to (169.0, 106.6)
- moved SW_RESET1 31.1 mm to (174.1, 111.2)
- moved C:0_CLOCK1 31.0 mm to (144.8, 103.9)
- moved C:1_CLOCK2 31.0 mm to (136.7, 103.9)
- moved Y_CLOCK1 31.0 mm to (140.9, 103.9)
- moved D10:5 4.76 mm to (267.5, 70.6)
- moved D10:6 4.76 mm to (248.4, 70.6)
- moved D10:9 4.76 mm to (191.3, 70.6)
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Routing:
- net COL2: track 676.0 -> 0.00 mm, vias 56 -> 0
- net COL0: track 604.0 -> 0.00 mm, vias 12 -> 0
- net COL1: track 597.9 -> 0.00 mm, vias 60 -> 0
- net COL4: track 523.2 -> 0.00 mm, vias 42 -> 0
- net COL3: track 522.8 -> 0.00 mm, vias 46 -> 0
- net COL5: track 488.4 -> 0.00 mm, vias 38 -> 0
- net COL6: track 428.9 -> 0.00 mm, vias 26 -> 0
- net COL7: track 346.0 -> 0.00 mm, vias 22 -> 0
- net +5V: track 328.5 -> 0.00 mm, vias 8 -> 0
- net COL8: track 297.8 -> 0.00 mm, vias 18 -> 0
- net COL9: track 265.0 -> 0.00 mm, vias 10 -> 0
- net GND: track 260.0 -> 0.00 mm, vias 6 -> 0
- net ROW4: track 232.6 -> 0.00 mm, vias 2 -> 0
- net ROW7: track 211.1 -> 0.00 mm
- net ROW3: track 201.1 -> 0.00 mm, vias 2 -> 0
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
Commit message: Footprint fixes
Parts:
- MX5:0_NU0: footprint MX_Alps_Hybrid:MX-2U-NoLED -> MX_Alps_Hybrid:MX-2U-ReversedStabilizers-NoLED
- MX5:9_SPC1: footprint MX_Alps_Hybrid:MX-6.25U-NoLED -> MX_Alps_Hybrid:MX-6.25U-ReversedStabilizers-NoLED

Commit message: Traced switches
Parts:
- MX0:0_AFT1: value MX-NoLED -> AFT
- MX0:1_PLAY1: value MX-NoLED -> PLAYPAUSE
- MX0:2_FWD1: value MX-NoLED -> FWD
- MX0:3_MUT1: value MX-NoLED -> MUTE
- MX0:4_VOL-1: value MX-NoLED -> VOLUP
- MX0:5_VOL+1: value MX-NoLED -> VOLDN
- MX0:6_ESC1: value MX-NoLED -> ESC
- MX0:7_F1: value MX-NoLED -> F1
- MX0:8_F2: value MX-NoLED -> F2
- MX0:9_F3, MX6:9_F4: value MX-NoLED -> F3
- MX10:0_PGU1: value MX-NoLED -> PAGE DOWN
- MX10:1_UP1: value MX-NoLED -> UP
- MX10:4_RSH1: value MX-NoLED -> RIGHT SHIFT
- MX10:5_/1: value MX-NoLED -> / ?
- MX10:6_.1: value MX-NoLED -> . >
- MX10:7_,1: value MX-NoLED -> , <
- MX10:8_M1: value MX-NoLED -> M
- MX10:9_N1: value MX-NoLED -> N
- MX11:0_RGT1: value MX-NoLED -> RIGHT
- MX11:1_DWN1: value MX-NoLED -> DOWN
- MX11:2_LFT1: value MX-NoLED -> LEFT
- MX11:3_RCT1: value MX-NoLED -> RIGHT CONTROL
- MX11:4_MEN1: value MX-NoLED -> MENU
- MX11:5_OS1: value MX-NoLED -> RIGHT WIN
- MX11:6_AGR1: value MX-NoLED -> RIGHT ALT
- MX1:0_NUM1: value MX-NoLED -> NUMLOK
- MX1:1_NU/1: value MX-NoLED -> NUM /
- MX1:2_NU*1: value MX-NoLED -> NUM *
- MX1:3_NU-1: value MX-NoLED -> NUM -
- MX1:4_TIL1: value MX-NoLED -> `
- MX1:5_1: value MX-NoLED -> 1
- MX1:6_2: value MX-NoLED -> 2
- MX1:7_3: value MX-NoLED -> 3
- MX1:8_4: value MX-NoLED -> 4
- MX1:9_5: value MX-NoLED -> 5
- MX2:0_NU7: value MX-NoLED -> NUM 7
- MX2:1_NU8: value MX-NoLED -> NUM 8
- MX2:2_NU9: value MX-NoLED -> NUM 9
- MX2:3_NU+1: value MX-NoLED -> NUM +
- MX2:4_TAB1: value MX-NoLED -> TAB
- MX2:5_Q1: value MX-NoLED -> Q
- MX2:6_W1: value MX-NoLED -> W
- MX2:7_E1: value MX-NoLED -> E
- MX2:8_R1: value MX-NoLED -> R
- MX2:9_T1: value MX-NoLED -> T
- MX3:0_NU4: value MX-NoLED -> NUM 4
- MX3:1_NU5: value MX-NoLED -> NUM 5
- MX3:2_NU6: value MX-NoLED -> NUM 6
- MX3:4_CAP1: value MX-NoLED -> CAPS
- MX3:5_A1: value MX-NoLED -> A
- MX3:6_S1: value MX-NoLED -> S
- MX3:7_D1: value MX-NoLED -> D
- MX3:8_F1: value MX-NoLED -> F
- MX3:9_G1: value MX-NoLED -> G
- MX4:0_NU1: value MX-NoLED -> NUM 1
- MX4:1_NU2: value MX-NoLED -> NUM 2
- MX4:2_NU3: value MX-NoLED -> NUM 3
- MX4:3_NEN1: value MX-NoLED -> NUM ENTER
- MX4:4_LSH1: value MX-NoLED -> LEFT SHIFT
- MX4:5_Z1: value MX-NoLED -> Z
- MX4:6_X1: value MX-NoLED -> X
- MX4:7_C1: value MX-NoLED -> C
- MX4:8_V1: value MX-NoLED -> V
- MX4:9_B1: value MX-NoLED -> B
- MX5:0_NU0: value MX-NoLED -> NUM 0
- MX5:2_NUD1: value MX-NoLED -> NUM DEL
- MX5:3_LCT1: value MX-NoLED -> LEFT CONTROL
- MX5:4_OS1: value MX-NoLED -> LEFT WIN
- MX5:5_LAL1: value MX-NoLED -> LEFT ALT
- MX5:9_SPC1: value MX-NoLED -> SPACE
- MX6:0_PRT1: value MX-NoLED -> PRT
- MX6:1_F12: value MX-NoLED -> F12
- MX6:2_F11: value MX-NoLED -> F11
- MX6:3_F10: value MX-NoLED -> F10
- MX6:4_F9: value MX-NoLED -> F9
- MX6:5_F8: value MX-NoLED -> F8
- MX6:6_F7: value MX-NoLED -> F7
- MX6:7_F6: value MX-NoLED -> F6
- MX6:8_F5: value MX-NoLED -> F5
- MX7:0_HOM1: value MX-NoLED -> HOME
- MX7:1_INS1: value MX-NoLED -> INS
- MX7:2_BSP1: value MX-NoLED -> BACKSPACE
- MX7:3_=1: value MX-NoLED -> = +
- MX7:4_-1: value MX-NoLED -> - (
- MX7:5_0: value MX-NoLED -> 0
- MX7:6_9: value MX-NoLED -> 9
- MX7:7_8: value MX-NoLED -> 8
- MX7:8_7: value MX-NoLED -> 7
- MX7:9_6: value MX-NoLED -> 6
- MX8:0_END1: value MX-NoLED -> END
- MX8:1_DEL1: value MX-NoLED -> DELETE
- MX8:2_\1: value MX-NoLED -> \ |
- MX8:3_]1: value MX-NoLED -> ] }
- MX8:4_[1: value MX-NoLED -> [ {
- MX8:5_P1: value MX-NoLED -> P
- MX8:6_O1: value MX-NoLED -> O
- MX8:7_I1: value MX-NoLED -> I
- MX8:8_U1: value MX-NoLED -> U
- MX8:9_Y1: value MX-NoLED -> Y
- MX9:0_PGU1: value MX-NoLED -> PAGE UP
- MX9:1_SLK1: value MX-NoLED -> SCROLL LOCK
- MX9:2_PUS1: value MX-NoLED -> PAUSE
- MX9:3_ENT1: value MX-NoLED -> ENTER
- MX9:4_'1: value MX-NoLED -> ' "
- MX9:5_;1: value MX-NoLED -> ; :
- MX9:6_L1: value MX-NoLED -> L
- MX9:7_K1: value MX-NoLED -> K
- MX9:8_J1: value MX-NoLED -> J
- MX9:9_H1: value MX-NoLED -> H
- moved SW_RESET1 60.0 mm to (126.1, 75.1)
- moved FUSE_USB1 53.4 mm to (114.9, -23.1), turned to 180 degrees
- moved R_D-1 52.7 mm to (123.6, -25.9), turned to 180 degrees
- moved R_D+1 51.4 mm to (123.6, -28.6), turned to 180 degrees
- moved R_RESET1 47.5 mm to (131.7, 77.2)
- moved USB1 38.7 mm to (108.2, -37.6)
- moved C:DCP1 34.6 mm to (136.1, 77.5)
- moved C_UCAP1 34.6 mm to (135.6, 82.2)
- moved C:DCP0 34.6 mm to (154.3, 79.3)
- moved C:DCP2 34.6 mm to (148.4, 92.1)
- moved CONT1 34.6 mm to (145.0, 83.1)
- moved C:DCP3 34.6 mm to (141.1, 92.1)
- moved R:HWB1 34.6 mm to (154.4, 88.0)
- moved C:1_CLOCK2 31.8 mm to (140.3, 72.3)
- moved Y_CLOCK1 31.8 mm to (144.5, 72.3)
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Routing:
- net COL2: track 0.00 -> 697.7 mm, vias 0 -> 8
- net COL0: track 0.00 -> 609.2 mm
- net COL1: track 0.00 -> 537.1 mm
- net COL3: track 0.00 -> 505.5 mm, vias 0 -> 4
- net COL4: track 0.00 -> 488.8 mm, vias 0 -> 2
- net COL5: track 0.00 -> 438.0 mm, vias 0 -> 3
- net COL6: track 0.00 -> 406.3 mm, vias 0 -> 4
- net COL7: track 0.00 -> 320.4 mm, vias 0 -> 4
- net COL8: track 0.00 -> 281.6 mm, vias 0 -> 4
- net COL9: track 0.00 -> 247.8 mm, vias 0 -> 4
- net ROW9: track 0.00 -> 245.2 mm, vias 0 -> 4
- net ROW4: track 0.00 -> 221.5 mm
- net ROW5: track 0.00 -> 195.5 mm
- net ROW7: track 0.00 -> 194.1 mm
- net ROW2: track 0.00 -> 193.9 mm
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
Commit message: Tracing complete. Added outlines
Parts:
- MX0:0_AFT1: value AFT -> MX-NoLED
- MX0:1_PLAY1: value PLAYPAUSE -> MX-NoLED
- MX0:2_FWD1: value FWD -> MX-NoLED
- MX0:3_MUT1: value MUTE -> MX-NoLED
- MX0:4_VOL-1: value VOLUP -> MX-NoLED
- MX0:5_VOL+1: value VOLDN -> MX-NoLED
- MX0:6_ESC1: value ESC -> MX-NoLED
- MX0:7_F1: value F1 -> MX-NoLED
- MX0:8_F2: value F2 -> MX-NoLED
- MX0:9_F3, MX6:9_F4: value F3 -> MX-NoLED
- MX10:0_PGU1: value PAGE DOWN -> MX-NoLED
- MX10:1_UP1: value UP -> MX-NoLED
- MX10:4_RSH1: value RIGHT SHIFT -> MX-NoLED
- MX10:5_/1: value / ? -> MX-NoLED
- MX10:6_.1: value . > -> MX-NoLED
- MX10:7_,1: value , < -> MX-NoLED
- MX10:8_M1: value M -> MX-NoLED
- MX10:9_N1: value N -> MX-NoLED
- MX11:0_RGT1: value RIGHT -> MX-NoLED
- MX11:1_DWN1: value DOWN -> MX-NoLED
- MX11:2_LFT1: value LEFT -> MX-NoLED
- MX11:3_RCT1: value RIGHT CONTROL -> MX-NoLED
- MX11:4_MEN1: value MENU -> MX-NoLED
- MX11:5_OS1: value RIGHT WIN -> MX-NoLED
- MX11:6_AGR1: value RIGHT ALT -> MX-NoLED
- MX1:0_NUM1: value NUMLOK -> MX-NoLED
- MX1:1_NU/1: value NUM / -> MX-NoLED
- MX1:2_NU*1: value NUM * -> MX-NoLED
- MX1:3_NU-1: value NUM - -> MX-NoLED
- MX1:4_TIL1: value ` -> MX-NoLED
- MX1:5_1: value 1 -> MX-NoLED
- MX1:6_2: value 2 -> MX-NoLED
- MX1:7_3: value 3 -> MX-NoLED
- MX1:8_4: value 4 -> MX-NoLED
- MX1:9_5: value 5 -> MX-NoLED
- MX2:0_NU7: value NUM 7 -> MX-NoLED
- MX2:1_NU8: value NUM 8 -> MX-NoLED
- MX2:2_NU9: value NUM 9 -> MX-NoLED
- MX2:3_NU+1: value NUM + -> MX-NoLED
- MX2:4_TAB1: value TAB -> MX-NoLED
- MX2:5_Q1: value Q -> MX-NoLED
- MX2:6_W1: value W -> MX-NoLED
- MX2:7_E1: value E -> MX-NoLED
- MX2:8_R1: value R -> MX-NoLED
- MX2:9_T1: value T -> MX-NoLED
- MX3:0_NU4: value NUM 4 -> MX-NoLED
- MX3:1_NU5: value NUM 5 -> MX-NoLED
- MX3:2_NU6: value NUM 6 -> MX-NoLED
- MX3:4_CAP1: value CAPS -> MX-NoLED
- MX3:5_A1: value A -> MX-NoLED
- MX3:6_S1: value S -> MX-NoLED
- MX3:7_D1: value D -> MX-NoLED
- MX3:8_F1: value F -> MX-NoLED
- MX3:9_G1: value G -> MX-NoLED
- MX4:0_NU1: value NUM 1 -> MX-NoLED
- MX4:1_NU2: value NUM 2 -> MX-NoLED
- MX4:2_NU3: value NUM 3 -> MX-NoLED
- MX4:3_NEN1: value NUM ENTER -> MX-NoLED
- MX4:4_LSH1: value LEFT SHIFT -> MX-NoLED
- MX4:5_Z1: value Z -> MX-NoLED
- MX4:6_X1: value X -> MX-NoLED
- MX4:7_C1: value C -> MX-NoLED
- MX4:8_V1: value V -> MX-NoLED
- MX4:9_B1: value B -> MX-NoLED
- MX5:0_NU0: value NUM 0 -> MX-NoLED
- MX5:2_NUD1: value NUM DEL -> MX-NoLED
- MX5:3_LCT1: value LEFT CONTROL -> MX-NoLED
- MX5:4_OS1: value LEFT WIN -> MX-NoLED
- MX5:5_LAL1: value LEFT ALT -> MX-NoLED
- MX5:9_SPC1: value SPACE -> MX-NoLED
- MX6:0_PRT1: value PRT -> MX-NoLED
- MX6:1_F12: value F12 -> MX-NoLED
- MX6:2_F11: value F11 -> MX-NoLED
- MX6:3_F10: value F10 -> MX-NoLED
- MX6:4_F9: value F9 -> MX-NoLED
- MX6:5_F8: value F8 -> MX-NoLED
- MX6:6_F7: value F7 -> MX-NoLED
- MX6:7_F6: value F6 -> MX-NoLED
- MX6:8_F5: value F5 -> MX-NoLED
- MX7:0_HOM1: value HOME -> MX-NoLED
- MX7:1_INS1: value INS -> MX-NoLED
- MX7:2_BSP1: value BACKSPACE -> MX-NoLED
- MX7:3_=1: value = + -> MX-NoLED
- MX7:4_-1: value - ( -> MX-NoLED
- MX7:5_0: value 0 -> MX-NoLED
- MX7:6_9: value 9 -> MX-NoLED
- MX7:7_8: value 8 -> MX-NoLED
- MX7:8_7: value 7 -> MX-NoLED
- MX7:9_6: value 6 -> MX-NoLED
- MX8:0_END1: value END -> MX-NoLED
- MX8:1_DEL1: value DELETE -> MX-NoLED
- MX8:2_\1: value \ | -> MX-NoLED
- MX8:3_]1: value ] } -> MX-NoLED
- MX8:4_[1: value [ { -> MX-NoLED
- MX8:5_P1: value P -> MX-NoLED
- MX8:6_O1: value O -> MX-NoLED
- MX8:7_I1: value I -> MX-NoLED
- MX8:8_U1: value U -> MX-NoLED
- MX8:9_Y1: value Y -> MX-NoLED
- MX9:0_PGU1: value PAGE UP -> MX-NoLED
- MX9:1_SLK1: value SCROLL LOCK -> MX-NoLED
- MX9:2_PUS1: value PAUSE -> MX-NoLED
- MX9:3_ENT1: value ENTER -> MX-NoLED
- MX9:4_'1: value ' " -> MX-NoLED
- MX9:5_;1: value ; : -> MX-NoLED
- MX9:6_L1: value L -> MX-NoLED
- MX9:7_K1: value K -> MX-NoLED
- MX9:8_J1: value J -> MX-NoLED
- MX9:9_H1: value H -> MX-NoLED
- moved R_D+1 35.3 mm to (113.7, 5.33), turned to 90 degrees
- moved R_D-1 33.7 mm to (111.0, 5.37), turned to 90 degrees
- moved FUSE_USB1 23.4 mm to (109.6, -0.38), turned to 90 degrees
- moved USB1 19.1 mm to (112.6, -19.1)
- moved C:DCP1 16.1 mm to (150.1, 69.5), turned to 45 degrees
- moved R_RESET1 14.5 mm to (144.7, 70.6), turned to 225 degrees
- moved C:DCP3 12.9 mm to (137.9, 79.6), turned to 225 degrees
- moved C:1_CLOCK2 12.7 mm to (152.9, 71.1), turned to 225 degrees
- moved Y_CLOCK1 11.4 mm to (155.7, 73.8), turned to 135 degrees
- moved C_UCAP1 10.4 mm to (142.2, 74.2), turned to 135 degrees
- moved C:0_CLOCK1 10.3 mm to (158.0, 76.1), turned to 225 degrees
- moved SW_RESET1 9.24 mm to (127.8, 84.2)
- moved C:DCP0 6.29 mm to (158.8, 83.7), turned to 45 degrees
- moved D4:8 5.88 mm to (153.5, 64.8)
- moved R:HWB1 4.88 mm to (150.6, 91.1), turned to 45 degrees
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Connections:
- CONT1 pad 10: Net-(CONT1-Pad10) -> ROW0
- CONT1 pad 11: Net-(CONT1-Pad11) -> ROW1
- CONT1 pad 12: Net-(CONT1-Pad12) -> ROW6
- CONT1 pad 18: Net-(CONT1-Pad18) -> ROW8
- CONT1 pad 19: Net-(CONT1-Pad19) -> ROW9
- CONT1 pad 20: Net-(CONT1-Pad20) -> ROW10
- CONT1 pad 21: Net-(CONT1-Pad21) -> ROW7
- CONT1 pad 22: Net-(CONT1-Pad22) -> COL1
- CONT1 pad 25: Net-(CONT1-Pad25) -> COL0
- CONT1 pad 26: Net-(CONT1-Pad26) -> COL2
- CONT1 pad 27: Net-(CONT1-Pad27) -> COL3
- CONT1 pad 28: Net-(CONT1-Pad28) -> ROW2
- CONT1 pad 29: Net-(CONT1-Pad29) -> ROW3
- CONT1 pad 30: Net-(CONT1-Pad30) -> ROW4
- CONT1 pad 31: Net-(CONT1-Pad31) -> ROW5
- CONT1 pad 32: Net-(CONT1-Pad32) -> ROW11
- CONT1 pad 36: Net-(CONT1-Pad36) -> COL9
- CONT1 pad 37: Net-(CONT1-Pad37) -> COL8
- CONT1 pad 38: Net-(CONT1-Pad38) -> COL7
- CONT1 pad 39: Net-(CONT1-Pad39) -> COL6
- CONT1 pad 40: Net-(CONT1-Pad40) -> COL5
- CONT1 pad 41: Net-(CONT1-Pad41) -> COL4
Routing:
- net GND: track 0.00 -> 212.8 mm
- net COL0: track 609.2 -> 813.9 mm, vias 0 -> 15
- net COL1: track 537.1 -> 719.4 mm, vias 0 -> 4
- net +5V: track 0.00 -> 181.6 mm, vias 0 -> 6
- net COL2: track 697.7 -> 870.8 mm, vias 8 -> 15
- net COL3: track 505.5 -> 663.7 mm, vias 4 -> 7
- net ROW0: track 173.2 -> 286.6 mm, vias 0 -> 8
- net COL4: track 488.8 -> 596.2 mm, vias 2 -> 3
- net ROW11: track 114.3 -> 212.7 mm, vias 0 -> 2
- net ROW6: track 171.4 -> 260.4 mm, vias 0 -> 6
- net Net-(CONT1-Pad3): track 0.00 -> 88.1 mm
- net Net-(CONT1-Pad4): track 0.00 -> 87.6 mm
- net ROW7: track 194.1 -> 280.5 mm, vias 0 -> 8
- net COL5: track 438.0 -> 522.0 mm, vias 3 -> 5
- net ROW2: track 193.9 -> 265.5 mm, vias 0 -> 6
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- added copper zone on B.Cu, net GND
Other:
- board size 399 x 117.7 mm -> 400.1 x 116.7 mm
