File: KeyboardPCB.kicad_pcb (KiCad board)
At the start: 2 copper layers, 400.1 x 118.5 mm, 236 parts

Commit message: finishing touches
Other:
- board text added: "MEDIA_MUTE"
- board text added: "MEDIA_VOLUP"
- board text removed: "MEDAI_MUTE"
- board text removed: "MEDAI_VOLUP"
Changed lines of the file:
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@@
-(kicad_pcb (version 20171130) (host pcbnew "(5.1.6)-1")
+(kicad_pcb (version 20171130) (host pcbnew "(5.1.4)-1")
   (general
     (thickness 1.6)
@@
       (drillshape 0)
       (scaleselection 1)
-      (outputdirectory "../Out/"))
+      (outputdirectory "./"))
   )
   (net 0 "")
@@
     (effects (font (size 1 1) (thickness 0.15)) (justify mirror))
   )
-  (gr_text MEDAI_VOLUP (at 65.024 -6.35) (layer B.SilkS)
+  (gr_text MEDIA_VOLUP (at 65.024 -6.35) (layer B.SilkS)
     (effects (font (size 1 1) (thickness 0.15)) (justify mirror))
   )
@@
     (effects (font (size 1 1) (thickness 0.15)) (justify mirror))
   )
-  (gr_text MEDAI_MUTE (at 26.924 -6.35) (layer B.SilkS)
+  (gr_text MEDIA_MUTE (at 26.924 -6.35) (layer B.SilkS)
     (effects (font (size 1 1) (thickness 0.15)) (justify mirror))
   )
